File: Power_Module/Power_Module.kicad_sch (KiCad schematic)
At the start: 1 part, among them Q1 AO3400A

Commit message: This is the changes for the motor controllers and the power module
Parts:
- added BT1, BT2: BH123A, BH123A:BAT_BH123A, symbol BH123A:BH123A
- added C1, C2: 100 nF, Capacitor_THT:C_Disc_D3.0mm_W2.0mm_P2.50mm, symbol Device:C_Small
- added D1, D2: 1N5817, Diode_THT:D_A-405_P7.62mm_Horizontal, symbol Device:D_Schottky
- added M1_Conn, M2_Conn: Conn_01x02_Pin, Connector_Wire:SolderWire-1.5sqmm_1x02_P6mm_D1.7mm_OD3mm, symbol Connector:Conn_01x02_Pin
- added M2_Trans: AO3400A, AO3400A:SOT95P280X125-3N, symbol AO3400A:AO3400A
- added PS1: TPS62162DSGR, TPS62162DSGR:SON50P200X200X80-9N, symbol TPS62162DSGR:TPS62162DSGR
- added R1, R3: 200 Ohm, Resistor_THT:R_Axial_DIN0204_L3.6mm_D1.6mm_P5.08mm_Horizontal, symbol Device:R
- added R2, R4: 10KOhm, Resistor_THT:R_Axial_DIN0204_L3.6mm_D1.6mm_P5.08mm_Horizontal, symbol Device:R
- renumbered Q1 to M1_Trans
Connections:
- net GND: now also BT1.N, M2_Trans.2, R2.1, R4.1
- net at M1_Trans.1: now also R1.2, R2.2
- net at M1_Trans.3: now also C1.1, D1.2 (A), M1_Conn.1 (Pin_1)
- new net: C2.1, D2.2 (A), M2_Conn.1 (Pin_1), M2_Trans.3
- new net: C2.2, D2.1 (K), M2_Conn.2 (Pin_2)
- new net: BT1.P, BT2.N
- new net: M2_Trans.1, R3.2, R4.2
- new net: C1.2, D1.1 (K), M1_Conn.2 (Pin_2)
- new net M1_GPIO: R1.1
- new net M2_GPIO: R3.1
- new net VDD: BT2.P
Other:
- note added: "Motor 1 Transistor"
- note added: "Motor 2 Transistor"
- note added: "Power"
- moved on the sheet: M1_Trans

Commit message: Board Final for check by Lum or Martin
Parts:
- removed M1_Trans, M2_Trans: AO3400A, AO3400A:SOT95P280X125-3N, symbol AO3400A:AO3400A
- added C3, C4, C5: 10uF, Capacitor_THT:C_Radial_D5.0mm_H5.0mm_P2.00mm, symbol Device:C
- added C6: 22uF, Capacitor_THT:C_Radial_D5.0mm_H5.0mm_P2.00mm, symbol Device:C
- added C7, C8, C9: 100 nF, Capacitor_THT:C_Disc_D3.0mm_W2.0mm_P2.50mm, symbol Device:C_Small
- added Fo_Conn1, Fo_Conn2: Conn_01x02_Pin, Connector_PinHeader_2.54mm:PinHeader_1x02_P2.54mm_Vertical, symbol Connector:Conn_01x02_Pin
- added L1: CVH252009-2R2M, CVH252009-2R2M:INDC2520X100N, symbol CVH252009-2R2M:CVH252009-2R2M
- added Q1, Q2: AO3400A, Package_TO_SOT_SMD:SOT-23_Handsoldering, symbol Transistor_FET:AO3400A
- added R5: 100k, Resistor_THT:R_Axial_DIN0204_L3.6mm_D1.6mm_P5.08mm_Horizontal, symbol Device:R
- added R6, R7: 10KOhm, Resistor_THT:R_Axial_DIN0204_L3.6mm_D1.6mm_P5.08mm_Horizontal, symbol Device:R
- added U1: SC0917, SC0917:MODULE_SC0917, symbol SC0917:SC0917
- M1_Conn1: renamed from M1_Conn; footprint Connector_Wire:SolderWire-1.5sqmm_1x02_P6mm_D1.7mm_OD3mm -> Connector_PinHeader_2.54mm:PinHeader_1x02_P2.54mm_Vertical
- M2_Conn1: renamed from M2_Conn; footprint Connector_Wire:SolderWire-1.5sqmm_1x02_P6mm_D1.7mm_OD3mm -> Connector_PinHeader_2.54mm:PinHeader_1x02_P2.54mm_Vertical
Connections:
- net GND: now also PS1.1 (PGND), PS1.4 (AGND), PS1.5 (FB), PS1.9 (EXP), C3.2, C4.2, C5.1, C6.2, C7.1, C8.1, C9.1, Q1.2 (S), Q2.2 (S), R6.2, R7.2, U1.13 (GND), U1.18 (GND), U1.23 (GND), U1.28 (GND), U1.3 (GND), U1.33 (AGND), U1.38 (GND), U1.8 (GND), U1.D2 (GND)
- net M1_GPIO: now also U1.26 (GP20)
- net M2_GPIO: now also U1.27 (GP21)
- net VDD: now also PS1.2 (VIN), PS1.3 (EN), C3.1, C4.1
- net at C2.1, D2.2 (A), M2_Conn1.1 (Pin_1): now also Q1.3 (D)
- net +3V3: now reaches C2.2, D2.1 (K), M2_Conn1.2 (Pin_2)
- net +3V3: now also C1.2, D1.1 (K), M1_Conn1.2 (Pin_2), PS1.6 (VOS), C5.2, C6.1, C7.2, C8.2, C9.2, Fo_Conn1.2 (Pin_2), Fo_Conn2.2 (Pin_2), L1.2, R5.1, U1.40 (VBUS)
- net at R3.2, R4.2: now also Q1.1 (G)
- net at R1.2, R2.2: now also Q2.1 (G)
- net at C1.1, D1.2 (A), M1_Conn1.1 (Pin_1): now also Q2.3 (D)
- net at PS1.7 (SW): now also L1.1
- net at PS1.8 (PG): now also R5.2
- new net Fo_Sens1: Fo_Conn1.1 (Pin_1), R6.1, U1.31 (GP26)
- new net Fo_Sens2: Fo_Conn2.1 (Pin_1), R7.1, U1.32 (GP27)
- new net USB_SHIELD: U1.A (USB_SHIELD), U1.B (USB_SHIELD), U1.C (USB_SHIELD), U1.D (USB_SHIELD)
Other:
- note added: "Controller"
- note added: "Force Sensors"
- moved on the sheet: BT1, C1, C2, D1, D2, M1_Conn1, M2_Conn1, PS1, R1, R2, R3, R4
